File: Keyboard_PCB.kicad_pcb (KiCad board)
At the start: 2 copper layers, 321 x 102 mm, 164 parts, among them J1 USB_C_Receptacle_USB2.0_16P, SW1 SW_Push, U1 USBLC6-2SC6, U2 MIC5365-3.3YC5, U3 STM32F401RCT6, Y1 25MHz, Y2 32kHz768

Commit message: Missing Matrix Connection to MCU
Parts:
- removed SW1: SW_Push, random-keyboard-parts.pretty-master:SKQG-1155865
- added J2: TC2030_SWD, Connector_IDC:IDC-Header_2x03_P2.54mm_Horizontal, B.Cu at (374.8, 143.4)
- added JP1: Jumper_2_Bridged, TestPoint:TestPoint_2Pads_Pitch2.54mm_Drill0.8mm, B.Cu at (370.5, 137.6)
- moved FB2 5.17 mm to (378.7, 127.4)
- moved C8 4.88 mm to (378.4, 130.8)
- moved C9 4.88 mm to (380.4, 130.8)
- moved C7 4.88 mm to (376.3, 130.8)
Routing:
- net NRST: track 6.49 -> 38.9 mm, vias 0 -> 2
- net SWDIO: track 0.00 -> 30.2 mm
- net SW0: track 0.00 -> 28.1 mm
- net SWCLK: track 0.00 -> 25.5 mm
- net BOOT0: track 38.8 -> 13.5 mm
- net COL01: track 63.2 -> 83.3 mm
- net COL14: track 85.1 -> 99.2 mm
- net +3V3: track 134.8 -> 146.2 mm, vias 8 -> 9
- net VDD: track 13.5 -> 23.2 mm, vias 0 -> 3
- net Net-(D59-A): track 0.00 -> 7.41 mm
- net Net-(D68-A): track 0.00 -> 6.62 mm
- net Net-(D67-A): track 0.00 -> 6.62 mm
- net Net-(D65-A): track 0.00 -> 6.62 mm
- net Net-(D64-A): track 0.00 -> 6.62 mm
- net Net-(D63-A): track 0.00 -> 6.62 mm
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
Commit message: PCB finished
Parts:
- moved C4 2.17 mm to (368.0, 109.2)
- moved D1 1.02 mm to (359.9, 108.6)
- moved R4 0.89 mm to (359.9, 111.0)
Connections:
- U3 pad 20: unconnected-(U3-PA4-Pad20) -> COL00
- U3 pad 21: unconnected-(U3-PA5-Pad21) -> COL01
- U3 pad 22: unconnected-(U3-PA6-Pad22) -> COL02
- U3 pad 23: unconnected-(U3-PA7-Pad23) -> COL03
- U3 pad 24: unconnected-(U3-PC4-Pad24) -> COL04
- U3 pad 25: unconnected-(U3-PC5-Pad25) -> COL05
- U3 pad 26: unconnected-(U3-PB0-Pad26) -> COL06
- U3 pad 27: unconnected-(U3-PB1-Pad27) -> COL07
- U3 pad 28: unconnected-(U3-PB2-Pad28) -> COL08
- U3 pad 29: unconnected-(U3-PB10-Pad29) -> COL09
- U3 pad 34: unconnected-(U3-PB13-Pad34) -> ROW0
- U3 pad 35: unconnected-(U3-PB14-Pad35) -> ROW1
- U3 pad 36: unconnected-(U3-PB15-Pad36) -> ROW2
- U3 pad 37: unconnected-(U3-PC6-Pad37) -> ROW3
- U3 pad 38: unconnected-(U3-PC7-Pad38) -> ROW4
- U3 pad 39: unconnected-(U3-PC8-Pad39) -> COL10
- U3 pad 40: unconnected-(U3-PC9-Pad40) -> COL11
- U3 pad 41: unconnected-(U3-PA8-Pad41) -> COL12
- U3 pad 42: unconnected-(U3-PA9-Pad42) -> COL13
- U3 pad 43: unconnected-(U3-PA10-Pad43) -> COL14
Routing:
- net COL00: track 76.4 -> 385.9 mm, vias 0 -> 8
- net COL01: track 83.3 -> 367.7 mm, vias 0 -> 8
- net COL02: track 82.3 -> 354.2 mm, vias 0 -> 6
- net COL03: track 63.2 -> 311.8 mm, vias 0 -> 6
- net COL04: track 63.2 -> 299.6 mm, vias 0 -> 4
- net COL05: track 63.2 -> 276.6 mm, vias 0 -> 4
- net COL06: track 83.2 -> 283.4 mm, vias 0 -> 2
- net COL07: track 63.2 -> 240.9 mm, vias 0 -> 2
- net COL08: track 63.2 -> 211.3 mm, vias 0 -> 2
- net COL10: track 89.7 -> 236.4 mm, vias 0 -> 3
- net COL11: track 94.4 -> 220.0 mm, vias 0 -> 3
- net COL09: track 86.2 -> 211.1 mm, vias 0 -> 2
- net COL12: track 84.4 -> 179.3 mm, vias 0 -> 3
- net COL13: track 83.2 -> 151.6 mm, vias 0 -> 3
- net ROW3: track 281.6 -> 344.7 mm, vias 0 -> 4
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
Commit message: save
Parts:
- added H1: MountingHole, MountingHole:MountingHole_2.2mm_M2, F.Cu at (385.8, 165.9)
- added H2: MountingHole, MountingHole:MountingHole_2.2mm_M2, F.Cu at (70.6, 165.9)
- added H3: MountingHole, MountingHole:MountingHole_2.2mm_M2, F.Cu at (70.6, 69.8)
- added H4: MountingHole, MountingHole:MountingHole_2.2mm_M2, F.Cu at (385.8, 69.8)
- added H5: MountingHole, MountingHole:MountingHole_2.2mm_M2, F.Cu at (165.9, 104.8)
- added H6: MountingHole, MountingHole:MountingHole_2.2mm_M2, F.Cu at (261.1, 105.6)
Routing:
- net COL14: track 105.5 -> 103.6 mm
